File: 808.brd (EAGLE design)
At the start: 160 x 100 mm, 56 parts, among them IC1 TL072D, T1 BC846, T2 BC846, T3 BC846, T5 BC846, T6 BC846

Commit message: regenerating brd
Parts:
- C8: value 0.47uF -> 0.47uF / 50v
- R19: value 10k -> 10k Log; device 808:POTENTIOMETER-3352P -> 808:POTENTIOMETER-PTV09
- R20: value 10k -> 100k Lin; device 808:POTENTIOMETER-3352P -> 808:POTENTIOMETER-CTS296
- R26: value 500k -> 500k Lin; device 808:POTENTIOMETER-3352P -> 808:POTENTIOMETER-PTV09
- T4: value (none) -> BC856
- moved S2 91.3 mm to (-24.1, 62.2)
- moved S1 88.6 mm to (-16.5, 62.2)
- moved C14 52.3 mm to (-36.8, 36.8)
- moved C13 50.0 mm to (-30.5, 36.8)
- moved R24 39.8 mm to (-16.5, 55.9)
- moved R27 39.8 mm to (-21.6, 55.9)
- moved C5 36.1 mm to (-24.1, 36.8)
- moved C10 36.1 mm to (-17.8, 36.8)
- moved R3 33.7 mm to (-16.5, 49.5)
- moved R7 33.7 mm to (-22.9, 49.5)
- moved IC1 31.4 mm to (-17.8, 20.3)
- moved T1 31.4 mm to (-26.7, 20.3)
- moved T4 29.9 mm to (-49.5, 20.3)
- moved R14 29.0 mm to (-29.2, 43.2)
- moved R5 29.0 mm to (-22.9, 43.2)
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
Commit message: layout
Parts:
- added J1: HEADER, Livestream:1X02-5.08-SCREWTERM
- added JP1: AUDIO-JACK-3P, Livestream:CUI-352X-SMT
- R19: value 10k Log -> Tone / 10k Log
- R20: value 100k Lin -> Level / 100k Lin
- R26: value 500k Lin -> Decay / 500k Lin
- moved R21 123.4 mm to (58.4, 23.6), turned to 180 degrees
- moved T6 117.0 mm to (52.1, 25.4), turned to 90 degrees
- moved R20 106.2 mm to (54.1, 7.62), turned to 180 degrees
- moved R23 102.2 mm to (58.4, 30.2), turned to 180 degrees
- moved R30 99.9 mm to (44.5, 30.5), turned to 90 degrees
- moved R22 99.7 mm to (55.3, 21.0)
- moved C12 97.8 mm to (52.1, 30.5)
- moved C7 95.9 mm to (33.0, 17.8), turned to 90 degrees
- moved R6 95.2 mm to (35.6, 34.3), turned to 270 degrees
- moved R18 92.5 mm to (29.2, 16.5), turned to 180 degrees
- moved C11 90.6 mm to (46.0, 18.1)
- moved R8 88.9 mm to (35.6, 22.9), turned to 270 degrees
- moved R9 88.3 mm to (19.1, 21.6), turned to 180 degrees
- moved C9 87.0 mm to (59.7, 19.1)
- moved D3 84.6 mm to (22.9, 11.4), turned to 90 degrees
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Connections:
- removed net VCC: C13.1, C14.2
- net +15V: now also C13.1, J1.P1
- net -15V: now also C14.2, J1.P2
- net GND: now also JP1.1
- net OUT: now also JP1.2, JP1.3
Routing:
- net +15V: track 0.00 -> 169.9 mm, vias 0 -> 5
- net -15V: track 0.00 -> 144.9 mm, vias 0 -> 4
- net GND: track 0.00 -> 56.4 mm, vias 0 -> 17
- net N$19: track 0.00 -> 53.9 mm, vias 0 -> 5
- net N$26: track 0.00 -> 36.6 mm, vias 0 -> 2
- net N$9: track 0.00 -> 29.5 mm, vias 0 -> 2
- net N$10: track 0.00 -> 27.1 mm
- net OUT: track 0.00 -> 25.8 mm
- net N$16: track 0.00 -> 22.1 mm, vias 0 -> 2
- net N$3: track 0.00 -> 17.1 mm
- net N$20: track 0.00 -> 16.1 mm
- net N$8: track 0.00 -> 14.4 mm
- net ACCENT: track 0.00 -> 12.9 mm
- net N$18: track 0.00 -> 12.0 mm
- net N$24: track 0.00 -> 11.2 mm
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- added copper zone on layer 16, net GND
Other:
- board size 160 x 100 mm -> 63.5 x 44.5 mm
- board text added: "+15V"
- board text added: "-15V"
- board text added: "6/14"
- board text added: "808 Kick v0.1"
- board text added: "Plover Electric"
