File: kick.sch (EAGLE design)
At the start: 58 parts, among them IC1 TL072D, J1 HEADER, T1 BC846, T2 BC846, T3 BC846, T4 BC856, T5 BC846, T6 BC846

Commit message: fixed some part numbers
Parts:
- R1, R6, R9: PARTNO RC2012F105CS -> RMCF0805FT1M00
- R10, R16: PARTNO RMCF0805JT4K70 -> RMCF0805FT4K70
- R11, R12, R18: PARTNO RC2012J103CS -> RMCF0805FT10K0
- R13, R28, R4: PARTNO RMCF0805JT22K0 -> RMCF0805FT22K0
- R14, R15, R22, R30, R5: PARTNO RC2012J104CS -> RMCF0805FT100K
- R17: PARTNO RMCF0805JT220R -> RMCF0805FT220R
- R2: PARTNO RMCF0805JT2K70 -> RMCF0805FT2K70
- R21: PARTNO RMCF0805JT82K0 -> RMCF0805FT82K0
- R24, R27, R8: PARTNO RMCF0805JT47K0 -> RMCF0805FT47K0
- R25: PARTNO RMCF0805JT470K -> CRCW0805470KFKEA
- R29: PARTNO RC2012J102CS -> RMCF0805FT1K00
- R3: PARTNO RMCF0805JT8K20 -> RMCF0805FT8K20
Changed lines of the file:
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@@
 <part name="SUPPLY1" library="supply2" deviceset="VCC" device="" value="+15V"/>
 <part name="R1" library="adafruit" deviceset="R-US_" device="R0805" value="1M">
-<attribute name="PARTNO" value="RC2012F105CS"/>
+<attribute name="PARTNO" value="RMCF0805FT1M00"/>
 </part>
 <part name="T1" library="transistor-neu-to92" deviceset="BC846" device="">
@@
 <part name="SUPPLY2" library="supply2" deviceset="GND" device=""/>
 <part name="R2" library="adafruit" deviceset="R-US_" device="R0805" value="2.7k">
-<attribute name="PARTNO" value="RMCF0805JT2K70"/>
+<attribute name="PARTNO" value="RMCF0805FT2K70"/>
 </part>
 <part name="SUPPLY3" library="supply2" deviceset="GND" device=""/>
 <part name="R3" library="adafruit" deviceset="R-US_" device="R0805" value="8.2k">
-<attribute name="PARTNO" value="RMCF0805JT8K20"/>
+<attribute name="PARTNO" value="RMCF0805FT8K20"/>
 </part>
 <part name="R4" library="adafruit" deviceset="R-US_" device="R0805" value="22k">
-<attribute name="PARTNO" value="RMCF0805JT22K0"/>
+<attribute name="PARTNO" value="RMCF0805FT22K0"/>
 </part>
 <part name="C2" library="adafruit" deviceset="C-US" device="C0805" value="33nF">
@@
 </part>
 <part name="R5" library="adafruit" deviceset="R-US_" device="R0805" value="100k">
-<attribute name="PARTNO" value="RC2012J104CS"/>
+<attribute name="PARTNO" value="RMCF0805FT100K"/>
 </part>
 <part name="R6" library="adafruit" deviceset="R-US_" device="R0805" value="1M">
-<attribute name="PARTNO" value="RC2012F105CS"/>
+<attribute name="PARTNO" value="RMCF0805FT1M00"/>
 </part>
 <part name="D1" library="adafruit" deviceset="DIODE" device="SOD-323F" value="1N4148">
@@
 </part>
 <part name="R8" library="adafruit" deviceset="R-US_" device="R0805" value="47k">
-<attribute name="PARTNO" value="RMCF0805JT47K0"/>
+<attribute name="PARTNO" value="RMCF0805FT47K0"/>
 </part>
 <part name="SUPPLY5" library="supply2" deviceset="GND" device=""/>
@@
 </part>
 <part name="R9" library="adafruit" deviceset="R-US_" device="R0805" value="1M">
-<attribute name="PARTNO" value="RC2012F105CS"/>
+<attribute name="PARTNO" value="RMCF0805FT1M00"/>
 </part>
 <part name="T4" library="transistor" deviceset="*-PNP-" device="SOT23-BEC" technology="BC856B" value="BC856">
@@
 </part>
 <part name="R10" library="adafruit" deviceset="R-US_" device="R0805" value="4.7k">
-<attribute name="PARTNO" value="RMCF0805JT4K70"/>
+<attribute name="PARTNO" value="RMCF0805FT4K70"/>
 </part>
 <part name="R11" library="adafruit" deviceset="R-US_" device="R0805" value="10k">
-<attribute name="PARTNO" value="RC2012J103CS"/>
+<attribute name="PARTNO" value="RMCF0805FT10K0"/>
 </part>
 <part name="T5" library="transistor-neu-to92" deviceset="BC846" device="">
@@
 <part name="SUPPLY6" library="supply2" deviceset="GND" device=""/>
 <part name="R12" library="adafruit" deviceset="R-US_" device="R0805" value="10k">
-<attribute name="PARTNO" value="RC2012J103CS"/>
+<attribute name="PARTNO" value="RMCF0805FT10K0"/>
 </part>
 <part name="R13" library="adafruit" deviceset="R-US_" device="R0805" value="22k">
-<attribute name="PARTNO" value="RMCF0805JT22K0"/>
+<attribute name="PARTNO" value="RMCF0805FT22K0"/>
 </part>
 <part name="C5" library="adafruit" deviceset="C-US" device="C0805" value="0.1uF">
@@
 </part>
 <part name="R14" library="adafruit" deviceset="R-US_" device="R0805" value="100k">
-<attribute name="PARTNO" value="RC2012J104CS"/>
+<attribute name="PARTNO" value="RMCF0805FT100K"/>
 </part>
 <part name="SUPPLY7" library="supply2" deviceset="GND" device=""/>
@@
 </part>
 <part name="R15" library="adafruit" deviceset="R-US_" device="R0805" value="100k">
-<attribute name="PARTNO" value="RC2012J104CS"/>
+<attribute name="PARTNO" value="RMCF0805FT100K"/>
 </part>
 <part name="R16" library="adafruit" deviceset="R-US_" device="R0805" value="4.7k">
-<attribute name="PARTNO" value="RMCF0805JT4K70"/>
+<attribute name="PARTNO" value="RMCF0805FT4K70"/>
 </part>
 <part name="SUPPLY8" library="supply2" deviceset="GND" device=""/>
@@
 </part>
 <part name="R17" library="adafruit" deviceset="R-US_" device="R0805" value="220R">
-<attribute name="PARTNO" value="RMCF0805JT220R"/>
+<attribute name="PARTNO" value="RMCF0805FT220R"/>
 </part>
 <part name="R18" library="adafruit" deviceset="R-US_" device="R0805" value="10k">
-<attribute name="PARTNO" value="RC2012J103CS"/>
+<attribute name="PARTNO" value="RMCF0805FT10K0"/>
 </part>
 <part name="C7" library="adafruit" deviceset="C-US" device="C0805" value="100nF">
@@
 </part>
 <part name="R21" library="adafruit" deviceset="R-US_" device="R0805" value="82k">
-<attribute name="PARTNO" value="RMCF0805JT82K0"/>
+<attribute name="PARTNO" value="RMCF0805FT82K0"/>
 </part>
 <part name="R22" library="adafruit" deviceset="R-US_" device="R0805" value="100k">
-<attribute name="PARTNO" value="RC2012J104CS"/>
+<attribute name="PARTNO" value="RMCF0805FT100K"/>
 </part>
 <part name="SUPPLY11" library="supply2" deviceset="GND" device=""/>
@@
 <part name="SUPPLY14" library="supply2" deviceset="VCC" device="" value="+15V"/>
 <part name="R24" library="adafruit" deviceset="R-US_" device="R0805" value="47k">
-<attribute name="PARTNO" value="RMCF0805JT47K0"/>
+<attribute name="PARTNO" value="RMCF0805FT47K0"/>
 </part>
 <part name="R25" library="adafruit" deviceset="R-US_" device="R0805" value="470k">
-<attribute name="PARTNO" value="RMCF0805JT470K"/>
+<attribute name="PARTNO" value="CRCW0805470KFKEA"/>
 </part>
 <part name="R26" library="808" deviceset="POT" device="PTV09-H" value="Decay / 500k Lin">
@@
 </part>
 <part name="R27" library="adafruit" deviceset="R-US_" device="R0805" value="47k">
-<attribute name="PARTNO" value="RMCF0805JT47K0"/>
+<attribute name="PARTNO" value="RMCF0805FT47K0"/>
 </part>
 <part name="R28" library="adafruit" deviceset="R-US_" device="R0805" value="22k">
-<attribute name="PARTNO" value="RMCF0805JT22K0"/>
+<attribute name="PARTNO" value="RMCF0805FT22K0"/>
 </part>
 <part name="SUPPLY15" library="supply2" deviceset="GND" device=""/>
@@
 </part>
 <part name="R29" library="adafruit" deviceset="R-US_" device="R0805" value="1k">
-<attribute name="PARTNO" value="RC2012J102CS"/>
+<attribute name="PARTNO" value="RMCF0805FT1K00"/>
 </part>
 <part name="R30" library="adafruit" deviceset="R-US_" device="R0805" value="100k">
-<attribute name="PARTNO" value="RC2012J104CS"/>
+<attribute name="PARTNO" value="RMCF0805FT100K"/>
 </part>
 <part name="SUPPLY16" library="supply2" deviceset="GND" device=""/>
