File: snare.brd (EAGLE design)
At the start: 160 x 100 mm, 76 parts, among them IC1 TL072D, IC2 TL072D, T1 BC846, T2 BC856, T3 BC846, T4 2N3704, T5 BC846, T6 BC846, T7 BC846

Commit message: snare layout
Parts:
- removed U$1: AUDIO-JACK-3P, Livestream:CUI-352X-SMT
- added JP1: HEADER, Livestream:1X02-5.08-SCREWTERM
- added JP2: AUDIO-JACK-3P, Livestream:CUI-352X-SMT
- S3: value TRIGGER -> ACCENT
- moved R34 129.3 mm to (51.3, 6.43)
- moved C24 113.7 mm to (46.4, 8.89), turned to 90 degrees
- moved T6 113.1 mm to (53.3, 8.89), turned to 270 degrees
- moved R33 112.2 mm to (38.7, 12.1), turned to 90 degrees
- moved T7 112.1 mm to (43.8, 5.08)
- moved C21 107.2 mm to (52.1, 12.1), turned to 90 degrees
- moved R31 107.1 mm to (38.7, 8.89), turned to 90 degrees
- moved R32 107.0 mm to (33.7, 6.99)
- moved C23 106.8 mm to (42.5, 8.89), turned to 270 degrees
- moved R30 102.2 mm to (36.8, 8.89), turned to 270 degrees
- moved C22 102.0 mm to (42.5, 12.1), turned to 270 degrees
- moved C20 101.7 mm to (48.3, 8.89), turned to 270 degrees
- moved R19 97.9 mm to (29.2, 32.4)
- moved R38 96.4 mm to (46.4, 4.45), turned to 90 degrees
- moved R16 96.3 mm to (45.1, 21.6), turned to 90 degrees
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Connections:
- net +15V: now also JP1.P1
- net -15V: now also JP1.P2
- net GND: now also JP2.1; no longer U$1.1
- net N$24: now also JP2.2, JP2.3; no longer U$1.2, U$1.3
Routing:
- net +15V: track 0.00 -> 232.4 mm, vias 0 -> 7
- net -15V: track 0.00 -> 147.0 mm, vias 0 -> 3
- net NOISE: track 0.00 -> 86.6 mm
- net N$15: track 0.00 -> 45.3 mm
- net GND: track 0.00 -> 44.4 mm, vias 0 -> 19
- net N$19: track 0.00 -> 38.1 mm, vias 0 -> 1
- net N$6: track 0.00 -> 31.8 mm
- net N$10: track 0.00 -> 29.7 mm, vias 0 -> 2
- net N$24: track 0.00 -> 29.7 mm
- net N$17: track 0.00 -> 29.0 mm
- net N$18: track 0.00 -> 24.2 mm, vias 0 -> 2
- net N$21: track 0.00 -> 20.8 mm, vias 0 -> 2
- net N$23: track 0.00 -> 18.6 mm, vias 0 -> 2
- net N$28: track 0.00 -> 15.1 mm
- net N$26: track 0.00 -> 12.7 mm
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- added copper zone on layer 16, net GND
Other:
- board size 160 x 100 mm -> 58.4 x 48.3 mm
- board text added: "+15V"
- board text added: "-15V"
- board text added: "Plover"
- board text added: "Plover Electric TR808 Snare v0.1 6/2014"

Commit message: fixed some part numbers
Parts:
- R8: value 820R -> 820k
Changed lines of the file:
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@@
 6/2014</text>
 <text x="47" y="0.4" size="1.9304" layer="1" font="vector">Plover</text>
+<text x="56.5" y="21.7" size="1.778" layer="30" font="vector" rot="MR270">Plover</text>
 </plain>
 <attributes>
@@
 <attribute name="PARTNO" value="RMCF0805FT680R" x="3.975" y="31.115" size="1.778" layer="27" rot="R180" display="off"/>
 </element>
-<element name="R8" library="SparkFun-Resistors" package="0805" value="820R" x="7.25" y="32.985" smashed="yes">
+<element name="R8" library="SparkFun-Resistors" package="0805" value="820k" x="7.25" y="32.985" smashed="yes">
 <attribute name="NAME" x="5.888" y="33.8105" size="0.4064" layer="25"/>
 <attribute name="VALUE" x="7.234" y="31.788" size="0.4064" layer="27"/>
-<attribute name="PARTNO" value="RMCF0805FT820R" x="7.25" y="32.985" size="1.778" layer="27" display="off"/>
+<attribute name="PARTNO" value="RC0805FR-07820KL" x="7.25" y="32.985" size="1.778" layer="27" display="off"/>
 </element>
 <element name="C4" library="SparkFun-Capacitors" package="0805" value="47nF" x="24.13" y="20.955" smashed="yes">
