File: hihats.sch (EAGLE design)
At the start: 41 parts, among them T1 BC846, T10 BC846, T2 BC856, T3 BC846, T4 BC856, T5 BC846, T6 BC846, T7 BC846, T8 BC846, T9 BC846

Commit message: fixed sch and started layout
Parts:
- added C10, C18: 33uF / 6.3v, Livestream:CAP-POLPANASONIC_B-2
- added C11, C22, C3: 22nF, SparkFun-Capacitors:CAP0805
- added C12, C13, C4, C6, C7: 1.5nF, SparkFun-Capacitors:CAP0805
- added C14, C15, C28: 1nF, SparkFun-Capacitors:CAP0805
- added C16, C32: 470pF, SparkFun-Capacitors:CAP0805
- added C17, C9: 220pF, SparkFun-Capacitors:CAP0805
- added C19: 0.47uF, Livestream:CAP-POLPANASONIC_B-2
- added C20, C21: 0.1uF, SparkFun-Capacitors:CAP0805
- added C23, C24, C27: 18nF, SparkFun-Capacitors:CAP0805
- added C25, C26: 10nF, SparkFun-Capacitors:CAP0805
- added C29, C30: 3.3nF, SparkFun-Capacitors:CAP0805
- added C31: 2.2uF, SparkFun-Capacitors:CAP0805
- added C33: 10uF / 16v, Livestream:CAP-POLPANASONIC_B-2
- added C8: 470p, SparkFun-Capacitors:CAP0805
- added D1, D2: FDLL914A, semicon-smd-ipc:D-MLL-34
- added IC1, IC3: TL072D, linear:TL072D
- added IC2: 4584D, 45xx:4584D
- added IC4: 5V, SparkFun-PowerIC:V_REG_MIC52055V
- added J1: AUDIO-JACK-3P, Livestream:AUDIO-JACK-3P
- added R25: 2M, 808:POTTHUMB-3352
- added R26, R44: 33k, SparkFun-Resistors:RESISTOR0805-RES
- added R27, R28, R38, R39: 1M, SparkFun-Resistors:RESISTOR0805-RES
- added R29, R40: 100R, SparkFun-Resistors:RESISTOR0805-RES
- added R30, R41: 2.7k, SparkFun-Resistors:RESISTOR0805-RES
- added R31, R42: 68k, SparkFun-Resistors:RESISTOR0805-RES
- added R32, R43, R61: 22k, SparkFun-Resistors:RESISTOR0805-RES
- added R33: 39k, SparkFun-Resistors:RESISTOR0805-RES
- added R34, R45: 47k, SparkFun-Resistors:RESISTOR0805-RES
- added R35, R46: 470k, SparkFun-Resistors:RESISTOR0805-RES
- added R36, R47: 100k Lin, 808:POTCTS296
- added R37, R48: 1k, SparkFun-Resistors:RESISTOR0805-RES
- added R49: 300k, SparkFun-Resistors:RESISTOR0805-RES
- added R50, R56, R57, R58, R59, R60: 120k, SparkFun-Resistors:RESISTOR0805-RES
- added R51: 270k, SparkFun-Resistors:RESISTOR0805-RES
- added R52: 220k, SparkFun-Resistors:RESISTOR0805-RES
- added R53: 680k, SparkFun-Resistors:RESISTOR0805-RES
- added R54, R55: 560k, SparkFun-Resistors:RESISTOR0805-RES
- added R62: 82k, SparkFun-Resistors:RESISTOR0805-RES
- added R63: 550R, SparkFun-Resistors:RESISTOR0805-RES
- added T11, T12, T13, T14: BC846, transistor-neu-to92:BC846
- C5: value 6.8nF -> 22nF
Connections:
- removed net VCC: S2.1
- new net +5V: C31.1, IC2P.VDD, IC4.OUT
- new net N$26: C4.1, C6.1, D1.A, R26.2
- new net N$27: R16.2, R25.A, R25.S
- new net N$28: R27.1, R28.2
- new net N$29: C5.1, R28.1, T11.B
- new net N$31: R29.2, T11.E
- new net N$32: C3.1, D1.C, T11.C
- new net N$33: C6.2, C7.1, R30.2
- new net N$34: C7.2, R31.2, T12.B
- new net N$35: C8.1, R30.1, R32.2, T12.E
- new net N$36: C8.2, R33.1
- new net N$37: C10.-, C9.1, IC1A.-IN, R33.2, R35.1
- new net N$38: IC1A.+IN, R34.2
- new net N$39: C9.2, IC1A.OUT, R35.2, R36.A, R36.S, R37.1
- new net N$40: R40.2, T13.E
- new net N$41: C10.+, R36.E
- new net N$42: C12.1, D2.C, T13.C
- new net N$43: R38.2, R39.1
- new net N$44: C11.1, R38.1, T13.B
- new net N$45: C13.1, C14.1, D2.A, R23.2
- new net N$46: C14.2, C15.1, R41.2
- new net N$47: C15.2, R42.2, T14.B
- new net N$48: C16.1, R41.1, R43.2, T14.E
- new net N$49: C16.2, R44.1
- new net N$50: C17.1, C18.-, IC1B.-IN, R44.2, R46.1
- new net N$51: IC1B.+IN, R45.2
- new net N$52: J1.LEFT, R37.2
- new net N$53: C17.2, IC1B.OUT, R46.2, R47.A, R47.S, R48.1
- new net N$54: C18.+, R47.E
- new net N$55: J1.RIGHT, R48.2
- new net N$56: IC2A.O, R49.2, R50.1
- new net N$57: C22.2, IC2A.I, R49.1
- new net N$58: C27.2, IC2F.I, R55.1
- new net N$59: C26.2, IC2E.I, R54.1
- new net N$60: C25.2, IC2D.I, R53.1
- new net N$61: C24.2, IC2C.I, R52.1
- new net N$62: C23.2, IC2B.I, R51.1
- new net N$63: IC2B.O, R51.2, R56.1
- new net N$64: IC2C.O, R52.2, R57.1
- new net N$65: IC2D.O, R53.2, R58.1
- new net N$66: IC2E.O, R54.2, R59.1
- new net N$67: IC2F.O, R55.2, R60.1
- new net N$68: C28.1, R50.2, R56.2, R57.2, R58.2, R59.2, R60.2
- new net N$69: IC3B.-IN, IC3B.OUT
- new net N$70: C28.2, R61.1
- new net N$71: C29.1, IC3A.-IN, R61.2, R62.1
- new net N$72: C29.2, C30.1, R63.2
- new net N$74: C32.1, IC4.BP
- new net NOISE: C11.2, C30.2, C5.2, IC3A.OUT, R62.2
- net +15V: now also C20.1, IC1P.V+, IC3P.V+, IC4.EN, IC4.IN, R25.E, R27.2, R39.2, S2.1, T12.C, T14.C
- net -15V: now also C21.1, IC1P.V-, IC3P.V-, R32.1, R43.1
- net GND: now also C12.2, C13.2, C19.-, C20.2, C21.2, C22.1, C23.1, C24.1, C25.1, C26.1, C27.1, C3.2, C31.2, C32.2, C33.-, C4.2, IC2P.VSS, IC3A.+IN, IC3B.+IN, IC4.GND, J1.SLEEVE, R29.1, R31.1, R34.1, R40.1, R42.1, R45.1, R63.1
- net N$16: now also R15.1, T7.C, T8.C; no longer R15.2, T5.E
- net N$17: now also C33.+
- net N$20: now also R26.1
- net N$22: now also R15.2, T5.E; no longer R15.1, T7.C, T8.C
- net N$24: now also C19.+

Commit message: bom for hats, combined bom
Parts:
- C1: PARTNO (none) -> EEE-1HAR47AR
- C10, C18: PARTNO (none) -> EEE-1AA330WAR
- C19: PARTNO (none) -> UWJ1HR47MCL1GB
- C2: PARTNO (none) -> EEE-1CA470WR
- C33: PARTNO (none) -> EEE-1VA100WAR
- D1, D2: PARTNO (none) -> FDLL914A
- IC1, IC3: PARTNO (none) -> TL072SG-13
- IC2: PARTNO (none) -> BU4584BF-E2
- IC4: PARTNO (none) -> MIC5205-5.0YM5 TR
- J1: PARTNO (none) -> SJ-3523-SMT-TR
- R25: PARTNO (none) -> 3352P-1-205LF
- R36, R47: PARTNO (none) -> 296UD104B1N
